Commit message: edit momonga

File: turtlebot3_description/urdf/turtlebot3_waffle.urdf.xacro (robot description, xacro)
@@ -140,5 +140,5 @@
     <parent link="base_link"/>
     <child link="base_scan"/>
-    <origin xyz="-0.064 0 0.122" rpy="0 0 0"/>
+    <origin xyz="-0.064 0 0.280" rpy="0 0 0"/>
   </joint>
   <link name="base_scan">
@@ -165,5 +165,5 @@
   </link>
   <joint name="camera_joint" type="fixed">
-    <origin xyz="0.064 -0.065 0.094" rpy="0 0 0"/>
+    <origin xyz="0.064 -0.065 0.115" rpy="0 0 0"/>
     <parent link="base_link"/>
     <child link="camera_link"/>

Commit message: edit camera link angle

File: turtlebot3_description/urdf/turtlebot3_waffle.urdf.xacro (robot description, xacro)
@@ -7,4 +7,5 @@
   <xacro:property name="r200_cam_rgb_pz" value="0.013"/>
   <xacro:property name="r200_cam_depth_offset" value="0.01"/>
+  <property name="M_PI" value="3.14159274"/>
   <link name="base_footprint"/>
   <joint name="base_joint" type="fixed">
@@ -165,5 +166,5 @@
   </link>
   <joint name="camera_joint" type="fixed">
-    <origin xyz="0.064 -0.065 0.115" rpy="0 0 0"/>
+    <origin xyz="0.064 -0.065 0.115" rpy="0 ${-10*M_PI/180} 0"/>
     <parent link="base_link"/>
     <child link="camera_link"/>

Commit message: edit camera joint angle for D435

File: turtlebot3_description/urdf/turtlebot3_waffle.urdf.xacro (robot description, xacro)
@@ -166,5 +166,5 @@
   </link>
   <joint name="camera_joint" type="fixed">
-    <origin xyz="0.064 -0.065 0.115" rpy="0 ${-10*M_PI/180} 0"/>
+    <origin xyz="0.064 -0.065 0.115" rpy="0 ${-7.7*M_PI/180} 0"/>
     <parent link="base_link"/>
     <child link="camera_link"/>

Commit message: edit D435 urdf setting

File: turtlebot3_description/urdf/turtlebot3_waffle.urdf.xacro (robot description, xacro)
@@ -166,5 +166,5 @@
   </link>
   <joint name="camera_joint" type="fixed">
-    <origin xyz="0.064 -0.065 0.115" rpy="0 ${-7.7*M_PI/180} 0"/>
+    <origin xyz="0.100 0 0.133" rpy="0 ${-7.7*M_PI/180} 0"/>
     <parent link="base_link"/>
     <child link="camera_link"/>
@@ -174,11 +174,11 @@
      <origin xyz="0 0 0" rpy="1.57 0 1.57"/>
       <geometry>
-       <mesh filename="package://turtlebot3_description/meshes/sensors/r200.dae" />
-      </geometry>
-    </visual>
-    <collision>
-      <origin xyz="0.003 0.065 0.007" rpy="0 0 0"/>
-      <geometry>
-        <box size="0.012 0.132 0.020"/>
+       <mesh filename="package://realsense2_camera/meshes/d435.dae" />
+      </geometry>
+    </visual>
+    <collision>
+      <origin xyz="0 0 0" rpy="0 0 0"/>
+      <geometry>
+        <box size="0.025 0.090 0.025"/>
       </geometry>
     </collision>
@@ -192,4 +192,5 @@
     </inertial>-->
   </link>
+<!--
   <joint name="camera_rgb_joint" type="fixed">
     <origin xyz="${r200_cam_rgb_px} ${r200_cam_rgb_py} ${r200_cam_rgb_pz}" rpy="0 0 0"/>
@@ -216,3 +217,4 @@
   </joint>
   <link name="camera_depth_optical_frame"/>
+-->
 </robot>
